File: lmx9838_1.brd (EAGLE design)
At the start: 37.4 x 43.6 mm, 34 parts, among them X1 MINI USB

Commit message: Bug Fixes Rev 2.0
Parts:
- moved U1 0.90 mm to (1.78, 7.37)
Routing:
- net GND: track 75.9 -> 78.1 mm
- net VDD: track 24.9 -> 25.8 mm
